File: STATUS_INDICATORS.kicad_sch (KiCad schematic)
At the start: 0 parts

Commit message: Autosave
Other:
- note added: "We need: 3x THT LEDs, various colors, with THT resistors 1x THT Buzzer, 5V rated"
Changed lines of the file:
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@@
 	(generator_version "10.0")
 	(paper "A4")
+	(text "We need:\n3x THT LEDs, various colors, with THT resistors\n1x THT Buzzer, 5V rated"
+		(exclude_from_sim no)
+		(at 74.168 65.786 0)
+		(effects
+			(font
+				(size 1.27 1.27)
+			)
+		)
+	)
 )
