File: EXTERNAL_CONNECTORS.kicad_sch (KiCad schematic)
At the start: 9 parts, among them CN4 DT15-12PA, CN5 DT15-12PA, CN6 DT15-12PA

Commit message: Autosave
Parts:
- CN4: Name POWER -> POWER/ENGINE2
Changed lines of the file:
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@@
 			)
 		)
-		(property "Name" "POWER"
-			(at 73.406 100.584 0)
+		(property "Name" "POWER/ENGINE2"
+			(at 69.342 100.584 0)
 			(show_name no)
 			(do_not_autoplace no)

Commit message: Autosave
Connections:
- net EXT_IN_SIG_BRAKE_PRESSURE_REAR: now also CN4.9; no longer CN4.11
- net EXT_IN_SIG_NEUTRAL_SAFETY: now also CN4.10; no longer CN4.12
Changed lines of the file:
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@@
+		)
+	)
+	(text "22AWG\n"
+		(exclude_from_sim no)
+		(at 89.154 91.694 0)
+		(effects
+			(font
+				(size 1.143 1.143)
+			)
 		)
 	)
@@
 		)
 	)
-	(text "22AWG\n"
-		(exclude_from_sim no)
-		(at 89.154 86.614 0)
-		(effects
-			(font
-				(size 1.143 1.143)
-			)
-		)
-	)
 	(text "16AWG\n"
 		(exclude_from_sim no)
@@
 	(text "22AWG\n"
 		(exclude_from_sim no)
-		(at 89.154 84.074 0)
-		(effects
-			(font
-				(size 1.143 1.143)
-			)
-		)
-	)
-	(text "22AWG\n"
-		(exclude_from_sim no)
 		(at 138.176 99.314 0)
 		(effects
@@
 		(exclude_from_sim no)
 		(at 138.176 89.154 0)
+		(effects
+			(font
+				(size 1.143 1.143)
+			)
+		)
+	)
+	(text "22AWG\n"
+		(exclude_from_sim no)
+		(at 89.154 89.154 0)
 		(effects
 			(font
@@
 	(wire
 		(pts
-			(xy 92.71 82.55) (xy 85.09 82.55)
-		)
-		(stroke
-			(width 0)
-			(type default)
-		)
-	)
-	(wire
-		(pts
 			(xy 127 116.84) (xy 127 115.57)
 		)
@@
 	(wire
 		(pts
+			(xy 92.71 90.17) (xy 85.09 90.17)
+		)
+		(stroke
+			(width 0)
+			(type default)
+		)
+	)
+	(wire
+		(pts
 			(xy 87.63 115.57) (xy 86.36 115.57)
 		)
@@
 	(wire
 		(pts
+			(xy 92.71 87.63) (xy 85.09 87.63)
+		)
+		(stroke
+			(width 0)
+			(type default)
+		)
+	)
+	(wire
+		(pts
 			(xy 185.42 115.57) (xy 185.42 116.84)
 		)
@@
 		(pts
 			(xy 87.63 127) (xy 86.36 127)
-		)
-		(stroke
-			(width 0)
-			(type default)
-		)
-	)
-	(wire
-		(pts
-			(xy 92.71 85.09) (xy 85.09 85.09)
 		)
 		(stroke
@@
 		)
 	)
+	(label "EXT_IN_SIG_NEUTRAL_SAFETY"
+		(at 92.71 87.63 0)
+		(effects
+			(font
+				(size 1.27 1.27)
+			)
+			(justify left bottom)
+		)
+	)
 	(label "PWR_FRONT_LIGHTS"
 		(at 92.71 95.25 0)
@@
 		)
 	)
+	(label "EXT_IN_SIG_BRAKE_PRESSURE_REAR"
+		(at 92.71 90.17 0)
+		(effects
+			(font
+				(size 1.27 1.27)
+			)
+			(justify left bottom)
+		)
+	)
 	(label "GND"
 		(at 87.63 127 0)
@@
 		)
 	)
-	(label "EXT_IN_SIG_NEUTRAL_SAFETY"
-		(at 92.71 82.55 0)
-		(effects
-			(font
-				(size 1.27 1.27)
-			)
-			(justify left bottom)
-		)
-	)
 	(label "EXT_OUT_SIG_IGNITION"
 		(at 142.24 82.55 0)
@@
 		(effects
 			(font
-				(size 1.27 1.27)
-			)
-			(justify left bottom)
-		)
-	)
-	(label "EXT_IN_SIG_BRAKE_PRESSURE_REAR"
-		(at 92.71 85.09 0)
-		(effects
-			(font

Commit message: Autosave
Connections:
- net EXT_OUT_SIG_IGNITION: now also CN4.12; no longer CN5.12
- net EXT_OUT_SIG_INJECTOR: now also CN4.11; no longer CN5.11
- net EXT_IN_SIG_MAP: no longer names the net of CN5.10
Changed lines of the file:
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@@
-	(text "22AWG\n"
-		(exclude_from_sim no)
-		(at 138.176 84.074 0)
-		(effects
-			(font
-				(size 1.143 1.143)
-			)
-		)
-	)
 	(text "22AWG\n"
 		(exclude_from_sim no)
@@
 		)
 	)
+	(text "22AWG"
+		(exclude_from_sim no)
+		(at 88.646 86.614 0)
+		(effects
+			(font
+				(size 1.143 1.143)
+			)
+		)
+	)
 	(text "16AWG\n"
 		(exclude_from_sim no)
@@
 		)
 	)
+	(text "22AWG\n"
+		(exclude_from_sim no)
+		(at 88.646 84.074 0)
+		(effects
+			(font
+				(size 1.143 1.143)
+			)
+		)
+	)
 	(text "16AWG\n"
 		(exclude_from_sim no)
 		(at 88.646 109.728 0)
-		(effects
-			(font
-				(size 1.143 1.143)
-			)
-		)
-	)
-	(text "22AWG"
-		(exclude_from_sim no)
-		(at 138.176 86.614 0)
 		(effects
 			(font
@@
 	(wire
 		(pts
-			(xy 142.24 85.09) (xy 134.62 85.09)
-		)
-		(stroke
-			(width 0)
-			(type default)
-		)
-	)
-	(wire
-		(pts
 			(xy 134.62 102.87) (xy 142.24 102.87)
 		)
@@
 	(wire
 		(pts
+			(xy 92.71 85.09) (xy 85.09 85.09)
+		)
+		(stroke
+			(width 0)
+			(type default)
+		)
+	)
+	(wire
+		(pts
 			(xy 184.15 110.49) (xy 191.77 110.49)
 		)
@@
 	(wire
 		(pts
-			(xy 142.24 82.55) (xy 134.62 82.55)
-		)
-		(stroke
-			(width 0)
-			(type default)
-		)
-	)
-	(wire
-		(pts
 			(xy 127 127) (xy 127 124.46)
 		)
@@
 		(pts
 			(xy 186.69 127) (xy 185.42 127)
+		)
+		(stroke
+			(width 0)
+			(type default)
+		)
+	)
+	(wire
+		(pts
+			(xy 92.71 82.55) (xy 85.09 82.55)
 		)
 		(stroke
@@
 		)
 	)
+	(label "EXT_OUT_SIG_INJECTOR"
+		(at 92.71 85.09 0)
+		(effects
+			(font
+				(size 1.27 1.27)
+			)
+			(justify left bottom)
+		)
+	)
 	(label "GND"
 		(at 92.71 110.49 0)
@@
 		)
 	)
-	(label "EXT_OUT_SIG_INJECTOR"
-		(at 142.24 85.09 0)
-		(effects
-			(font
-				(size 1.27 1.27)
-			)
-			(justify left bottom)
-		)
-	)
 	(label "GND"
 		(at 137.16 127 0)
@@
 		)
 	)
-	(label "EXT_IN_SIG_MAP"
-		(at 142.24 87.63 0)
-		(effects
-			(font
-				(size 1.27 1.27)
-			)
-			(justify left bottom)
-		)
-	)
 	(label "GND"
 		(at 186.69 127 0)
@@
 		)
 	)
-	(label "EXT_OUT_SIG_IGNITION"
-		(at 142.24 82.55 0)
-		(effects
-			(font
-				(size 1.27 1.27)
-			)
-			(justify left bottom)
-		)
-	)
 	(label "PWR_FUEL_PUMP"
 		(at 92.71 105.41 0)
@@
 		(effects
 			(font
+				(size 1.27 1.27)
+			)
+			(justify left bottom)
+		)
+	)
+	(label "EXT_OUT_SIG_IGNITION"
+		(at 92.71 82.55 0)
+		(effects
+			(font

Commit message: Autosave
Connections:
- net EXT_IN_SIG_RPM+: no longer CN5.6
Changed lines of the file:
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@@
-		)
-	)
-	(label "EXT_IN_SIG_RPM+"
-		(at 142.24 97.79 0)
-		(effects
-			(font
-				(size 1.27 1.27)
-			)
-			(justify left bottom)
 		)
 	)
@@
 	)
 	(label "EXT_IN_SIG_RPM-"
-		(at 134.62 77.47 0)
+		(at 147.32 82.55 0)
 		(effects
 			(font
@@
 		)
 	)
+	(label "EXT_IN_SIG_RPM+"
+		(at 147.32 85.09 0)
+		(effects
+			(font
+				(size 1.27 1.27)
+			)
+			(justify left bottom)
+		)
+	)
 	(label "EXT_IN_SIG_NEUTRAL_SAFETY"
 		(at 92.71 87.63 0)
@@
 		)
 	)
+	(label "EXT_IN_SIG_COOLANT_TEMP"
+		(at 129.54 72.39 0)
+		(effects
+			(font
+				(size 1.27 1.27)
+			)
+			(justify left bottom)
+		)
+	)
+	(label "EXT_IN_SIG_THROTTLE_POSITION"
+		(at 129.54 74.93 0)
+		(effects
+			(font
+				(size 1.27 1.27)
+			)
+			(justify left bottom)
+		)
+	)
 	(label "PWR_FUEL_PUMP"
 		(at 92.71 105.41 0)
 		(effects
 			(font
+				(size 1.27 1.27)
+			)
+			(justify left bottom)
+		)
+	)
+	(label "EXT_IN_SIG_INTAKE_TEMP"
+		(at 129.54 69.85 0)
+		(effects
+			(font

Commit message: Autosave
Connections:
- net EXT_IN_SIG_COOLANT_TEMP: now also CN5.7; no longer CN5.8
- net EXT_IN_SIG_INTAKE_TEMP: now also CN5.8; no longer CN5.9
- net EXT_IN_SIG_THROTTLE_POSITION: now also CN5.6; no longer CN5.7
Changed lines of the file:
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@@
-		)
-	)
-	(label "EXT_IN_SIG_COOLANT_TEMP"
-		(at 142.24 92.71 0)
-		(effects
-			(font
-				(size 1.27 1.27)
-			)
-			(justify left bottom)
 		)
 	)
@@
 	)
 	(label "EXT_IN_SIG_COOLANT_TEMP"
-		(at 129.54 72.39 0)
+		(at 142.24 95.25 0)
 		(effects
 			(font
@@
 	)
 	(label "EXT_IN_SIG_THROTTLE_POSITION"
-		(at 129.54 74.93 0)
+		(at 142.24 97.79 0)
 		(effects
 			(font
@@
 	)
 	(label "EXT_IN_SIG_INTAKE_TEMP"
-		(at 129.54 69.85 0)
+		(at 142.24 92.71 0)
 		(effects
 			(font
@@
 		)
 	)
-	(label "EXT_IN_SIG_THROTTLE_POSITION"
-		(at 142.24 95.25 0)
-		(effects
-			(font
-				(size 1.27 1.27)
-			)
-			(justify left bottom)
-		)
-	)
 	(label "EXT_OUT_SIG_IGNITION"
 		(at 92.71 82.55 0)
 		(effects
 			(font
-				(size 1.27 1.27)
-			)
-			(justify left bottom)
-		)
-	)
-	(label "EXT_IN_SIG_INTAKE_TEMP"
-		(at 142.24 90.17 0)
-		(effects
-			(font

Commit message: Autosave
Connections:
- net EXT_OUT_SIG_IGNITION: now also CN5.10
- net EXT_OUT_SIG_INJECTOR: now also CN5.9
Changed lines of the file:
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@@
+		)
+	)
+	(label "EXT_OUT_SIG_IGNITION"
+		(at 142.24 87.63 0)
+		(effects
+			(font
+				(size 1.27 1.27)
+			)
+			(justify left bottom)
 		)
 	)
@@
 		(effects
 			(font
+				(size 1.27 1.27)
+			)
+			(justify left bottom)
+		)
+	)
+	(label "EXT_OUT_SIG_INJECTOR"
+		(at 142.24 90.17 0)
+		(effects
+			(font

Commit message: Autosave
Connections:
- net EXT_IN_SIG_COOLANT_TEMP: now also CN5.9; no longer CN5.7
- net EXT_IN_SIG_INTAKE_TEMP: now also CN5.10; no longer CN5.8
- net EXT_IN_SIG_RPM+: now also CN5.6
- net EXT_IN_SIG_RPM-: now also CN5.7
- net EXT_IN_SIG_THROTTLE_POSITION: now also CN5.8; no longer CN5.6
- net EXT_OUT_SIG_IGNITION: no longer CN5.10
- net EXT_OUT_SIG_INJECTOR: no longer CN5.9
Changed lines of the file:
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@@
+		)
+	)
+	(label "EXT_IN_SIG_INTAKE_TEMP"
+		(at 142.24 87.63 0)
+		(effects
+			(font
+				(size 1.27 1.27)
+			)
+			(justify left bottom)
 		)
 	)
@@
 	)
 	(label "EXT_IN_SIG_RPM-"
-		(at 147.32 82.55 0)
+		(at 142.24 95.25 0)
 		(effects
 			(font
@@
 	)
 	(label "EXT_IN_SIG_RPM+"
-		(at 147.32 85.09 0)
+		(at 142.24 97.79 0)
 		(effects
 			(font
@@
 	)
 	(label "EXT_IN_SIG_COOLANT_TEMP"
-		(at 142.24 95.25 0)
+		(at 142.24 90.17 0)
 		(effects
 			(font
@@
 	)
 	(label "EXT_IN_SIG_THROTTLE_POSITION"
-		(at 142.24 97.79 0)
-		(effects
-			(font
-				(size 1.27 1.27)
-			)
-			(justify left bottom)
-		)
-	)
-	(label "EXT_OUT_SIG_IGNITION"
-		(at 142.24 87.63 0)
+		(at 142.24 92.71 0)
 		(effects
 			(font
@@
 		)
 	)
-	(label "EXT_IN_SIG_INTAKE_TEMP"
-		(at 142.24 92.71 0)
-		(effects
-			(font
-				(size 1.27 1.27)
-			)
-			(justify left bottom)
-		)
-	)
 	(label "PWR_12V"
 		(at 142.24 107.95 0)
@@
 		(effects
 			(font
-				(size 1.27 1.27)
-			)
-			(justify left bottom)
-		)
-	)
-	(label "EXT_OUT_SIG_INJECTOR"
-		(at 142.24 90.17 0)
-		(effects
-			(font

Commit message: Autosave
Connections:
- net EXT_OUT_SIG_IGNITION: now also CN5.12; no longer CN4.12
- net EXT_OUT_SIG_INJECTOR: now also CN5.11; no longer CN4.11
- net EXT_IN_SIG_BRAKE_PRESSURE_REAR: no longer names the net of CN4.9
Changed lines of the file:
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@@
-		)
-	)
-	(text "22AWG\n"
-		(exclude_from_sim no)
-		(at 88.646 84.074 0)
-		(effects
-			(font
-				(size 1.143 1.143)
-			)
 		)
 	)
@@
 	(text "22AWG\n"
 		(exclude_from_sim no)
+		(at 138.176 84.074 0)
+		(effects
+			(font
+				(size 1.143 1.143)
+			)
+		)
+	)
+	(text "22AWG\n"
+		(exclude_from_sim no)
 		(at 138.176 99.314 0)
 		(effects
@@
 		(exclude_from_sim no)
 		(at 187.2848 91.694 0)
+		(effects
+			(font
+				(size 1.143 1.143)
+			)
+		)
+	)
+	(text "22AWG"
+		(exclude_from_sim no)
+		(at 138.176 86.614 0)
 		(effects
 			(font
@@
 	(wire
 		(pts
-			(xy 92.71 85.09) (xy 85.09 85.09)
-		)
-		(stroke
-			(width 0)
-			(type default)
-		)
-	)
-	(wire
-		(pts
 			(xy 184.15 110.49) (xy 191.77 110.49)
 		)
@@
 	(wire
 		(pts
+			(xy 142.24 82.55) (xy 134.62 82.55)
+		)
+		(stroke
+			(width 0)
+			(type default)
+		)
+	)
+	(wire
+		(pts
 			(xy 134.62 95.25) (xy 142.24 95.25)
 		)
@@
 	(wire
 		(pts
+			(xy 142.24 85.09) (xy 134.62 85.09)
+		)
+		(stroke
+			(width 0)
+			(type default)
+		)
+	)
+	(wire
+		(pts
 			(xy 85.09 102.87) (xy 92.71 102.87)
 		)
@@
 		(pts
 			(xy 186.69 127) (xy 185.42 127)
-		)
-		(stroke
-			(width 0)
-			(type default)
-		)
-	)
-	(wire
-		(pts
-			(xy 92.71 82.55) (xy 85.09 82.55)
 		)
 		(stroke
@@
 		)
 	)
+	(label "EXT_OUT_SIG_INJECTOR"
+		(at 142.24 85.09 0)
+		(effects
+			(font
+				(size 1.27 1.27)
+			)
+			(justify left bottom)
+		)
+	)
 	(label "PWR_12V"
 		(at 186.69 115.57 0)
@@
 		)
 	)
-	(label "EXT_OUT_SIG_INJECTOR"
-		(at 92.71 85.09 0)
-		(effects
-			(font
-				(size 1.27 1.27)
-			)
-			(justify left bottom)
-		)
-	)
 	(label "GND"
 		(at 92.71 110.49 0)
@@
 		)
 	)
+	(label "EXT_OUT_SIG_IGNITION"
+		(at 142.24 82.55 0)
+		(effects
+			(font
+				(size 1.27 1.27)
+			)
+			(justify left bottom)
+		)
+	)
 	(label "EXT_IN_SIG_DASH_BTN_ONE"
 		(at 190.5 87.63 0)
@@
 		)
 	)
-	(label "EXT_IN_SIG_BRAKE_PRESSURE_REAR"
-		(at 92.71 90.17 0)
-		(effects
-			(font
-				(size 1.27 1.27)
-			)
-			(justify left bottom)
-		)
-	)
 	(label "GND"
 		(at 87.63 127 0)
@@
 		(effects
 			(font
-				(size 1.27 1.27)
-			)
-			(justify left bottom)
-		)
-	)
-	(label "EXT_OUT_SIG_IGNITION"
-		(at 92.71 82.55 0)
-		(effects
-			(font
