File: EXTERNAL_CONNECTORS.kicad_sch (KiCad schematic)
At the start: 9 parts, among them CN4 DT15-12PA, CN5 DT15-12PA, CN6 DT15-12PA

Commit message: Autosave
Connections:
- net EXT_IN_SIG_BRAKE_PRESSURE_REAR: now also CN4.11; no longer CN4.9
- net EXT_IN_SIG_COOLANT_TEMP: now also CN5.8; no longer CN5.9
- net EXT_IN_SIG_INTAKE_TEMP: now also CN5.9; no longer CN5.10
- net EXT_IN_SIG_NEUTRAL_SAFETY: now also CN4.12; no longer CN4.10
- net EXT_IN_SIG_RPM-: no longer CN5.7
- net EXT_IN_SIG_THROTTLE_POSITION: now also CN5.7; no longer CN5.8
- new net EXT_IN_SIG_MAP: CN5.10

Commit message: Autosave
Parts:
- CN4: Name POWER/ENGINE2 -> POWER
Connections:
- net EXT_IN_SIG_RPM+ renamed EXT_IN_SIG_RPM
Changed lines of the file:
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@@
 	(text "EXT_IN_SIG_RPM"
 		(exclude_from_sim no)
-		(at 168.402 70.612 0)
+		(at 156.972 74.93 0)
 		(effects
 			(font
@@
 		)
 	)
-	(label "EXT_IN_SIG_RPM+"
+	(label "EXT_IN_SIG_RPM"
 		(at 142.24 97.79 0)
 		(effects
@@
 	(label "GND"
 		(at 92.71 110.49 0)
-		(effects
-			(font
-				(size 1.27 1.27)
-			)
-			(justify left bottom)
-		)
-	)
-	(label "EXT_IN_SIG_RPM-"
-		(at 134.62 77.47 0)
 		(effects
 			(font
@@
 			)
 		)
-		(property "Name" "POWER/ENGINE2"
+		(property "Name" "POWER"
 			(at 73.406 100.584 0)
 			(show_name no)

Commit message: Autosave
Connections:
- net EXT_IN_SIG_COOLANT_TEMP: no longer CN5.8
- net EXT_IN_SIG_INTAKE_TEMP: no longer CN5.9
- net EXT_IN_SIG_MAP: no longer CN5.10
- net EXT_IN_SIG_THROTTLE_POSITION: no longer CN5.7
- net EXT_OUT_SIG_IGNITION: no longer CN5.12
- net EXT_OUT_SIG_INJECTOR: no longer CN5.11
Other:
- note removed: "EXT_IN_SIG_RPM"
Changed lines of the file:
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@@
-		)
-	)
-	(text "EXT_IN_SIG_RPM"
-		(exclude_from_sim no)
-		(at 156.972 74.93 0)
-		(effects
-			(font
-				(size 1.27 1.27)
-			)
 		)
 	)
@@
 		)
 	)
-	(label "EXT_IN_SIG_COOLANT_TEMP"
-		(at 142.24 92.71 0)
+	(label "EXT_IN_SIG_MAP"
+		(at 138.43 66.04 0)
 		(effects
 			(font
@@
 		)
 	)
+	(label "EXT_IN_SIG_THROTTLE_POSITION"
+		(at 138.43 73.66 0)
+		(effects
+			(font
+				(size 1.27 1.27)
+			)
+			(justify left bottom)
+		)
+	)
 	(label "EXT_IN_ESTOP_SIG_RETURN"
 		(at 190.5 82.55 0)
@@
 		)
 	)
+	(label "EXT_OUT_SIG_IGNITION"
+		(at 138.43 60.96 0)
+		(effects
+			(font
+				(size 1.27 1.27)
+			)
+			(justify left bottom)
+		)
+	)
 	(label "PWR_REAR_LIGHTS"
 		(at 92.71 97.79 0)
@@
 		)
 	)
-	(label "EXT_OUT_SIG_INJECTOR"
-		(at 142.24 85.09 0)
-		(effects
-			(font
-				(size 1.27 1.27)
-			)
-			(justify left bottom)
-		)
-	)
 	(label "GND"
 		(at 137.16 127 0)
@@
 		)
 	)
-	(label "EXT_IN_SIG_MAP"
-		(at 142.24 87.63 0)
-		(effects
-			(font
-				(size 1.27 1.27)
-			)
-			(justify left bottom)
-		)
-	)
 	(label "GND"
 		(at 186.69 127 0)
@@
 		)
 	)
+	(label "EXT_IN_SIG_INTAKE_TEMP"
+		(at 138.43 68.58 0)
+		(effects
+			(font
+				(size 1.27 1.27)
+			)
+			(justify left bottom)
+		)
+	)
 	(label "EXT_BI_SIG_CAN_HIGH"
 		(at 142.24 102.87 0)
@@
 		)
 	)
-	(label "EXT_OUT_SIG_IGNITION"
-		(at 142.24 82.55 0)
-		(effects
-			(font
-				(size 1.27 1.27)
-			)
-			(justify left bottom)
-		)
-	)
 	(label "PWR_FUEL_PUMP"
 		(at 92.71 105.41 0)
@@
 		)
 	)
-	(label "EXT_IN_SIG_THROTTLE_POSITION"
-		(at 142.24 95.25 0)
-		(effects
-			(font
-				(size 1.27 1.27)
-			)
-			(justify left bottom)
-		)
-	)
-	(label "EXT_IN_SIG_INTAKE_TEMP"
-		(at 142.24 90.17 0)
-		(effects
-			(font
+	(label "EXT_IN_SIG_COOLANT_TEMP"
+		(at 138.43 71.12 0)
+		(effects
+			(font
+				(size 1.27 1.27)
+			)
+			(justify left bottom)
+		)
+	)
+	(label "EXT_OUT_SIG_INJECTOR"
+		(at 138.43 63.5 0)
+		(effects
+			(font

Commit message: Autosave
Connections:
- net EXT_IN_SIG_RPM-: now reaches CN5.7
- net EXT_IN_SIG_RPM renamed EXT_IN_SIG_RPM+
Changed lines of the file:
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@@
 		)
 	)
-	(label "EXT_IN_SIG_RPM"
+	(label "EXT_IN_SIG_RPM+"
 		(at 142.24 97.79 0)
 		(effects
@@
 		(effects
 			(font
+				(size 1.27 1.27)
+			)
+			(justify left bottom)
+		)
+	)
+	(label "EXT_IN_SIG_RPM-"
+		(at 142.24 95.25 0)
+		(effects
+			(font

Commit message: Autosave
Connections:
- net EXT_IN_SIG_BRAKE_PRESSURE_REAR: no longer CN4.11
- net EXT_IN_SIG_COOLANT_TEMP: now also CN5.9
- net EXT_IN_SIG_INTAKE_TEMP: now also CN5.10
- net EXT_IN_SIG_MAP: now also CN5.11
- net EXT_IN_SIG_NEUTRAL_SAFETY: no longer CN4.12
- net EXT_IN_SIG_THROTTLE_POSITION: now also CN5.8
Changed lines of the file:
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@@
-		)
-	)
-	(text "22AWG\n"
-		(exclude_from_sim no)
-		(at 89.154 86.614 0)
-		(effects
-			(font
-				(size 1.143 1.143)
-			)
 		)
 	)
@@
 	(text "22AWG\n"
 		(exclude_from_sim no)
-		(at 89.154 84.074 0)
-		(effects
-			(font
-				(size 1.143 1.143)
-			)
-		)
-	)
-	(text "22AWG\n"
-		(exclude_from_sim no)
 		(at 138.176 99.314 0)
 		(effects
@@
 		(exclude_from_sim no)
 		(at 187.452 104.394 0)
+		(effects
+			(font
+				(size 1.143 1.143)
+			)
+		)
+	)
+	(text "22AWG\n"
+		(exclude_from_sim no)
+		(at 89.154 70.104 0)
+		(effects
+			(font
+				(size 1.143 1.143)
+			)
+		)
+	)
+	(text "22AWG\n"
+		(exclude_from_sim no)
+		(at 89.154 72.644 0)
 		(effects
 			(font
@@
 	(wire
 		(pts
-			(xy 92.71 82.55) (xy 85.09 82.55)
-		)
-		(stroke
-			(width 0)
-			(type default)
-		)
-	)
-	(wire
-		(pts
 			(xy 127 116.84) (xy 127 115.57)
 		)
@@
 	(wire
 		(pts
+			(xy 92.71 71.12) (xy 85.09 71.12)
+		)
+		(stroke
+			(width 0)
+			(type default)
+		)
+	)
+	(wire
+		(pts
 			(xy 86.36 127) (xy 77.47 127)
 		)
@@
 	(wire
 		(pts
+			(xy 92.71 68.58) (xy 85.09 68.58)
+		)
+		(stroke
+			(width 0)
+			(type default)
+		)
+	)
+	(wire
+		(pts
 			(xy 135.89 127) (xy 127 127)
 		)
@@
 	(wire
 		(pts
-			(xy 92.71 85.09) (xy 85.09 85.09)
-		)
-		(stroke
-			(width 0)
-			(type default)
-		)
-	)
-	(wire
-		(pts
 			(xy 142.24 90.17) (xy 134.62 90.17)
 		)
@@
 	)
 	(label "EXT_IN_SIG_MAP"
-		(at 138.43 66.04 0)
+		(at 142.24 85.09 0)
 		(effects
 			(font
@@
 	)
 	(label "EXT_IN_SIG_THROTTLE_POSITION"
-		(at 138.43 73.66 0)
+		(at 142.24 92.71 0)
 		(effects
 			(font
@@
 		)
 	)
+	(label "EXT_IN_SIG_BRAKE_PRESSURE_REAR"
+		(at 92.71 71.12 0)
+		(effects
+			(font
+				(size 1.27 1.27)
+			)
+			(justify left bottom)
+		)
+	)
 	(label "EXT_IN_SIG_STARTER"
 		(at 190.5 85.09 0)
@@
 	)
 	(label "EXT_IN_SIG_INTAKE_TEMP"
-		(at 138.43 68.58 0)
+		(at 142.24 87.63 0)
 		(effects
 			(font
@@
 		)
 	)
-	(label "EXT_IN_SIG_NEUTRAL_SAFETY"
-		(at 92.71 82.55 0)
-		(effects
-			(font
-				(size 1.27 1.27)
-			)
-			(justify left bottom)
-		)
-	)
 	(label "EXT_IN_SIG_RPM-"
 		(at 142.24 95.25 0)
@@
 		)
 	)
+	(label "EXT_IN_SIG_NEUTRAL_SAFETY"
+		(at 92.71 68.58 0)
+		(effects
+			(font
+				(size 1.27 1.27)
+			)
+			(justify left bottom)
+		)
+	)
 	(label "PWR_FUEL_PUMP"
 		(at 92.71 105.41 0)
@@
 		)
 	)
-	(label "EXT_IN_SIG_BRAKE_PRESSURE_REAR"
-		(at 92.71 85.09 0)
+	(label "EXT_IN_SIG_MAP"
+		(at 107.95 78.74 0)
 		(effects
 			(font
@@
 	)
 	(label "EXT_IN_SIG_COOLANT_TEMP"
-		(at 138.43 71.12 0)
-		(effects
-			(font
+		(at 142.24 90.17 0)
+		(effects
+			(font

Commit message: Autosave
Connections:
- net EXT_IN_SIG_BRAKE_PRESSURE_REAR: now also CN4.10
- net EXT_IN_SIG_NEUTRAL_SAFETY: now also CN4.11
Changed lines of the file:
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@@
+		)
+	)
+	(text "22AWG\n"
+		(exclude_from_sim no)
+		(at 87.884 70.104 0)
+		(effects
+			(font
+				(size 1.143 1.143)
+			)
 		)
 	)
@@
 	(text "22AWG\n"
 		(exclude_from_sim no)
-		(at 89.154 70.104 0)
-		(effects
-			(font
-				(size 1.143 1.143)
-			)
-		)
-	)
-	(text "22AWG\n"
-		(exclude_from_sim no)
-		(at 89.154 72.644 0)
+		(at 87.884 67.564 0)
+		(effects
+			(font
+				(size 1.143 1.143)
+			)
+		)
+	)
+	(text "22AWG\n"
+		(exclude_from_sim no)
+		(at 89.154 86.614 0)
+		(effects
+			(font
+				(size 1.143 1.143)
+			)
+		)
+	)
+	(text "22AWG\n"
+		(exclude_from_sim no)
+		(at 89.154 89.154 0)
 		(effects
 			(font
@@
 	(wire
 		(pts
+			(xy 91.44 66.04) (xy 83.82 66.04)
+		)
+		(stroke
+			(width 0)
+			(type default)
+		)
+	)
+	(wire
+		(pts
 			(xy 185.42 127) (xy 176.53 127)
 		)
@@
 	(wire
 		(pts
-			(xy 92.71 71.12) (xy 85.09 71.12)
+			(xy 92.71 87.63) (xy 85.09 87.63)
 		)
 		(stroke
@@
 	(wire
 		(pts
+			(xy 91.44 68.58) (xy 83.82 68.58)
+		)
+		(stroke
+			(width 0)
+			(type default)
+		)
+	)
+	(wire
+		(pts
 			(xy 185.42 115.57) (xy 185.42 116.84)
 		)
@@
 	(wire
 		(pts
-			(xy 92.71 68.58) (xy 85.09 68.58)
+			(xy 92.71 85.09) (xy 85.09 85.09)
 		)
 		(stroke
@@
 	)
 	(label "EXT_IN_SIG_BRAKE_PRESSURE_REAR"
-		(at 92.71 71.12 0)
+		(at 92.71 87.63 0)
 		(effects
 			(font
@@
 		)
 	)
+	(label "EXT_IN_SIG_BRAKE_PRESSURE_REAR"
+		(at 91.44 68.58 0)
+		(effects
+			(font
+				(size 1.27 1.27)
+			)
+			(justify left bottom)
+		)
+	)
 	(label "PWR_FRONT_LIGHTS"
 		(at 92.71 95.25 0)
@@
 		)
 	)
+	(label "EXT_IN_SIG_NEUTRAL_SAFETY"
+		(at 91.44 66.04 0)
+		(effects
+			(font
+				(size 1.27 1.27)
+			)
+			(justify left bottom)
+		)
+	)
 	(label "EXT_BI_SIG_CAN_HIGH"
 		(at 142.24 102.87 0)
@@
 	)
 	(label "EXT_IN_SIG_NEUTRAL_SAFETY"
-		(at 92.71 68.58 0)
-		(effects
-			(font
+		(at 92.71 85.09 0)
+		(effects
+			(font

Commit message: SCH Save
Connections:
- net EXT_IN_SIG_MAP: now also CN4.12
Changed lines of the file:
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@@
-		)
-	)
-	(text "22AWG\n"
-		(exclude_from_sim no)
-		(at 87.884 70.104 0)
-		(effects
-			(font
-				(size 1.143 1.143)
-			)
 		)
 	)
@@
 	(text "22AWG\n"
 		(exclude_from_sim no)
-		(at 87.884 67.564 0)
+		(at 89.154 84.074 0)
 		(effects
 			(font
@@
 	(wire
 		(pts
-			(xy 91.44 66.04) (xy 83.82 66.04)
+			(xy 92.71 82.55) (xy 85.09 82.55)
 		)
 		(stroke
@@
 		(pts
 			(xy 87.63 115.57) (xy 86.36 115.57)
-		)
-		(stroke
-			(width 0)
-			(type default)
-		)
-	)
-	(wire
-		(pts
-			(xy 91.44 68.58) (xy 83.82 68.58)
 		)
 		(stroke
@@
 		)
 	)
-	(label "EXT_IN_SIG_BRAKE_PRESSURE_REAR"
-		(at 91.44 68.58 0)
-		(effects
-			(font
-				(size 1.27 1.27)
-			)
-			(justify left bottom)
-		)
-	)
 	(label "PWR_FRONT_LIGHTS"
 		(at 92.71 95.25 0)
@@
 		)
 	)
-	(label "EXT_IN_SIG_NEUTRAL_SAFETY"
-		(at 91.44 66.04 0)
-		(effects
-			(font
-				(size 1.27 1.27)
-			)
-			(justify left bottom)
-		)
-	)
 	(label "EXT_BI_SIG_CAN_HIGH"
 		(at 142.24 102.87 0)
@@
 	)
 	(label "EXT_IN_SIG_MAP"
-		(at 107.95 78.74 0)
-		(effects
-			(font
+		(at 92.71 82.55 0)
+		(effects
+			(font

Commit message: SCH Save
Connections:
- net EXT_IN_SIG_MAP: no longer CN5.11
- net EXT_OUT_SIG_IGNITION: now also CN5.12
- net EXT_OUT_SIG_INJECTOR: now also CN5.11
Changed lines of the file:
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@@
-		)
-	)
-	(label "EXT_IN_SIG_MAP"
-		(at 142.24 85.09 0)
-		(effects
-			(font
-				(size 1.27 1.27)
-			)
-			(justify left bottom)
 		)
 	)
@@
 	)
 	(label "EXT_OUT_SIG_IGNITION"
-		(at 138.43 60.96 0)
+		(at 142.24 82.55 0)
 		(effects
 			(font
@@
 	)
 	(label "EXT_OUT_SIG_INJECTOR"
-		(at 138.43 63.5 0)
-		(effects
-			(font
+		(at 142.24 85.09 0)
+		(effects
+			(font
