File: ECU_INTERFACE.kicad_sch (KiCad schematic)
At the start: 0 parts

Commit message: SCH Save
Parts:
- added J10: 5569-16A2, Connector_Molex:Molex_Mini-Fit_Jr_5569-16A2_2x08_P4.20mm_Horizontal, symbol Connector_Generic:Conn_02x08_Top_Bottom
Changed lines of the file:
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@@
 	(generator_version "10.0")
 	(paper "A4")
+	(symbol
+		(lib_id "Connector_Generic:Conn_02x08_Top_Bottom")
+		(at 74.93 59.69 0)
+		(mirror x)
+		(unit 1)
+		(body_style 1)
+		(exclude_from_sim no)
+		(in_bom yes)
+		(on_board yes)
+		(in_pos_files yes)
+		(dnp no)
+		(property "Reference" "J10"
+			(at 76.2 46.99 0)
+			(show_name no)
+			(do_not_autoplace no)
+			(effects
+				(font
+					(size 1.27 1.27)
+				)
+			)
+		)
+		(property "Value" "5569-16A2"
+			(at 76.2 69.85 0)
+			(show_name no)
+			(do_not_autoplace no)
+			(effects
+				(font
+					(size 1.27 1.27)
+				)
+			)
+		)
+		(property "Footprint" "Connector_Molex:Molex_Mini-Fit_Jr_5569-16A2_2x08_P4.20mm_Horizontal"
+			(at 74.93 59.69 0)
+			(hide yes)
+			(show_name no)
+			(do_not_autoplace no)
+			(effects
+				(font
+					(size 1.27 1.27)
+				)
+			)
+		)
+		(property "Datasheet" ""
+			(at 74.93 59.69 0)
+			(hide yes)
+			(show_name no)
+			(do_not_autoplace no)
+			(effects
+				(font
+					(size 1.27 1.27)
+				)
+			)
+		)
+		(property "Description" ""
+			(at 74.93 59.69 0)
+			(hide yes)
+			(show_name no)
+			(do_not_autoplace no)
+			(effects
+				(font
+					(size 1.27 1.27)
+				)
+			)
+		)
+		(property "LCSC" "C485577"
+			(at 74.93 59.69 0)
+			(hide yes)
+			(show_name no)
+			(do_not_autoplace no)
+			(effects
+				(font
+					(size 1.27 1.27)
+				)
+			)
+		)
+		(pin "1"
+		)
+		(pin "10"
+		)
+		(pin "11"
+		)
+		(pin "12"
+		)
+		(pin "13"
+		)
+		(pin "14"
+		)
+		(pin "15"
+		)
+		(pin "16"
+		)
+		(pin "2"
+		)
+		(pin "3"
+		)
+		(pin "4"
+		)
+		(pin "5"
+		)
+		(pin "6"
+		)
+		(pin "7"
+		)
+		(pin "8"
+		)
+		(pin "9"
+		)
+		(instances
+			(project "Hub-2.0"
+				(path "/af8ad92e-80c5-47c7-b528-865d82af0364/92353b5a-0bb5-4764-8ad6-9a983b2830ec"
+					(reference "J10")
+					(unit 1)
+				)
+			)
+		)
+	)
 )

Commit message: Autosave
Changed lines of the file:
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@@
 	(symbol
 		(lib_id "Connector_Generic:Conn_02x08_Top_Bottom")
-		(at 74.93 59.69 0)
+		(at 66.04 54.61 0)
 		(mirror x)
 		(unit 1)
@@
 		(dnp no)
 		(property "Reference" "J10"
-			(at 76.2 46.99 0)
+			(at 67.31 41.91 0)
 			(show_name no)
 			(do_not_autoplace no)
@@
 		)
 		(property "Value" "5569-16A2"
-			(at 76.2 69.85 0)
+			(at 67.31 64.77 0)
 			(show_name no)
 			(do_not_autoplace no)
@@
 		)
 		(property "Footprint" "Connector_Molex:Molex_Mini-Fit_Jr_5569-16A2_2x08_P4.20mm_Horizontal"
-			(at 74.93 59.69 0)
+			(at 66.04 54.61 0)
 			(hide yes)
 			(show_name no)
@@
 		)
 		(property "Datasheet" ""
-			(at 74.93 59.69 0)
+			(at 66.04 54.61 0)
 			(hide yes)
 			(show_name no)
@@
 		)
 		(property "Description" ""
-			(at 74.93 59.69 0)
+			(at 66.04 54.61 0)
 			(hide yes)
 			(show_name no)
@@
 		)
 		(property "LCSC" "C485577"
-			(at 74.93 59.69 0)
+			(at 66.04 54.61 0)
 			(hide yes)
 			(show_name no)

Commit message: Autosave
Connections:
- net IN_AUX1: now reaches J10.1 (Pin_1)
- net IN_BUTTON2: now reaches J10.10 (Pin_10)
- net GNDA: now reaches J10.11 (Pin_11)
- net GNDA: now also J10.12 (Pin_12)
- net IN_TPS1: now reaches J10.13 (Pin_13)
- net IN_KNOCK_RAW: now reaches J10.14 (Pin_14)
- net IN_IAT: now reaches J10.15 (Pin_15)
- net IN_CLT: now reaches J10.16 (Pin_16)
- net IN_BUTTON1: now reaches J10.2 (Pin_2)
- net +5VP: now reaches J10.3 (Pin_3)
- net +5VP: now also J10.4 (Pin_4)
- net IN_FLEX: now reaches J10.5 (Pin_5)
- net IN_PPS1: now reaches J10.6 (Pin_6)
- net CAN+: now reaches J10.7 (Pin_7)
- net CAN-: now reaches J10.8 (Pin_8)
- net IN_MAP: now reaches J10.9 (Pin_9)
Other:
- note added: "D"

Commit message: Autosave
Parts:
- added J2: 5569-20A2, Connector_Molex:Molex_Mini-Fit_Jr_5569-20A2_2x10_P4.20mm_Horizontal, symbol Connector_Generic:Conn_02x10_Top_Bottom
Connections:
- net +5VP: now also J2.1 (Pin_1), J2.2 (Pin_2)
- net GNDA: now also J2.11 (Pin_11), J2.12 (Pin_12), J2.13 (Pin_13)
- new net EGT+: J2.10 (Pin_10)
- new net EGT-: J2.20 (Pin_20)
- new net GND: J2.8 (Pin_8)
- new net IN_AUX2: J2.3 (Pin_3)
- new net IN_AUX3: J2.15 (Pin_15)
- new net IN_BUTTON3: J2.9 (Pin_9)
- new net IN_HALL1: J2.5 (Pin_5)
- new net IN_HALL2: J2.6 (Pin_6)
- new net IN_HALL3: J2.7 (Pin_7)
- new net IN_PPS2: J2.4 (Pin_4)
- new net IN_TPS2: J2.14 (Pin_14)
- new net VR_DISCRETE+: J2.18 (Pin_18)
- new net VR_DISCRETE-: J2.19 (Pin_19)
- new net VR_MAX9924+: J2.16 (Pin_16)
- new net VR_MAX9924-: J2.17 (Pin_17)
Other:
- note added: "C"

Commit message: Autosave
Parts:
- added J5: 5569-18A2, Connector_Molex:Molex_Mini-Fit_Jr_5569-18A2_2x09_P4.20mm_Horizontal, symbol Connector_Generic:Conn_02x09_Top_Bottom
Connections:
- new net OUT_IGN1: J5.15 (Pin_15)
- new net OUT_IGN2: J5.14 (Pin_14)
- new net OUT_IGN3: J5.12 (Pin_12)
- new net OUT_IGN4: J5.11 (Pin_11)
- new net OUT_IGN5: J5.13 (Pin_13)
- new net OUT_IGN6: J5.10 (Pin_10)
- new net OUT_INJ1: J5.6 (Pin_6)
- new net OUT_INJ2: J5.5 (Pin_5)
- new net OUT_INJ3: J5.4 (Pin_4)
- new net OUT_INJ4: J5.3 (Pin_3)
- new net OUT_INJ5: J5.2 (Pin_2)
- new net OUT_INJ6: J5.1 (Pin_1)
- new net OUT_LS1: J5.7 (Pin_7)
- new net OUT_LS2: J5.18 (Pin_18)
- new net OUT_LS3: J5.17 (Pin_17)
- new net OUT_LS4: J5.16 (Pin_16)
- new net OUT_LS_HOT1: J5.9 (Pin_9)
- new net OUT_LS_HOT2: J5.8 (Pin_8)
Other:
- note added: "B"

Commit message: Autosave
Parts:
- added J4: 5569-08A2, Connector_Molex:Molex_Mini-Fit_Jr_5569-08A2_2x04_P4.20mm_Horizontal, symbol Connector_Generic:Conn_02x04_Top_Bottom
Connections:
- net GND: now also J4.3 (Pin_3), J4.4 (Pin_4)
- new net 12V_KEY: J4.7 (Pin_7)
- new net OUT_DC1+: J4.5 (Pin_5)
- new net OUT_DC1-: J4.1 (Pin_1)
- new net OUT_DC2+: J4.6 (Pin_6)
- new net OUT_DC2-: J4.2 (Pin_2)
Other:
- note added: "A"

Commit message: PCB Save
Parts:
- added J3: 5569-06A2, Connector_Molex:Molex_Mini-Fit_Jr_5569-06A2_2x03_P4.20mm_Horizontal, symbol Connector_Generic:Conn_02x03_Top_Bottom
Connections:
- new net +12V_RAW: J3.1 (Pin_1)
- new net 1_WBO_Ip: J3.5 (Pin_5)
- new net 2_WBO_Vm: J3.6 (Pin_6)
- new net 3_WBO_Heater: J3.3 (Pin_3)
- new net 5_WBO_Rtrim: J3.2 (Pin_2)
- new net 6_WBO_Un: J3.4 (Pin_4)
Other:
- note added: "E"

Commit message: Autosave
Connections:
- net CAN+ renamed ECU_CAN_HIGH
- net CAN- renamed ECU_CAN_LOW
Changed lines of the file:
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@@
 		)
 	)
-	(label "CAN+"
+	(label "ECU_CAN_HIGH"
 		(at 59.69 48.26 180)
 		(effects
@@
 		)
 	)
-	(label "CAN-"
+	(label "ECU_CAN_LOW"
 		(at 59.69 45.72 180)
 		(effects
