File: ECU_INTERFACE.kicad_sch (KiCad schematic)
At the start: 5 parts, among them J10 5569-16A2, J2 5569-20A2, J3 5569-06A2, J4 5569-08A2, J5 5569-18A2

Commit message: Autosave
Connections:
- net OUT_LS1 renamed ECU_OUT_LS1
- net OUT_LS_HOT1 renamed ECU_OUT_LS_HOT1
- net OUT_LS_HOT2 renamed ECU_OUT_LS_HOT2
Changed lines of the file:
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@@
 		)
 	)
-	(label "OUT_LS_HOT2"
+	(label "ECU_OUT_LS_HOT2"
 		(at 60.96 92.71 180)
 		(effects
@@
 		)
 	)
-	(label "OUT_LS_HOT1"
+	(label "ECU_OUT_LS_HOT1"
 		(at 60.96 90.17 180)
 		(effects
@@
 		)
 	)
-	(label "OUT_LS1"
+	(label "ECU_OUT_LS1"
 		(at 60.96 95.25 180)
 		(effects

Commit message: Autosave
Connections:
- net OUT_INJ1 renamed ECU_OUT_INJ1
- net OUT_INJ2 renamed ECU_OUT_INJ2
Changed lines of the file:
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@@
 		)
 	)
-	(label "OUT_INJ2"
+	(label "ECU_OUT_INJ2"
 		(at 60.96 100.33 180)
 		(effects
@@
 		)
 	)
-	(label "OUT_INJ1"
+	(label "ECU_OUT_INJ1"
 		(at 60.96 97.79 180)
 		(effects

Commit message: Autosave
Connections:
- net OUT_INJ3 renamed ECU_OUT_INJ3
- net OUT_INJ4 renamed ECU_OUT_INJ4
Changed lines of the file:
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@@
 		)
 	)
-	(label "OUT_INJ3"
+	(label "ECU_OUT_INJ3"
 		(at 60.96 102.87 180)
 		(effects
@@
 		)
 	)
-	(label "OUT_INJ4"
+	(label "ECU_OUT_INJ4"
 		(at 60.96 105.41 180)
 		(effects

Commit message: Autosave
Connections:
- net OUT_INJ5 renamed ECU_OUT_INJ5
Changed lines of the file:
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@@
 		)
 	)
-	(label "OUT_INJ5"
+	(label "ECU_OUT_INJ5"
 		(at 60.96 107.95 180)
 		(effects

Commit message: Autosave
Connections:
- net OUT_INJ6 renamed ECU_OUT_INJ6
- net OUT_LS2 renamed ECU_OUT_LS2
Changed lines of the file:
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@@
 		)
 	)
-	(label "OUT_INJ6"
+	(label "ECU_OUT_INJ6"
 		(at 60.96 110.49 180)
 		(effects
@@
 		)
 	)
-	(label "OUT_LS2"
+	(label "ECU_OUT_LS2"
 		(at 73.66 90.17 0)
 		(effects

Commit message: Autosave
Connections:
- net OUT_LS3 renamed ECU_OUT_LS3
- net OUT_LS4 renamed ECU_OUT_LS4
Changed lines of the file:
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@@
 		)
 	)
-	(label "OUT_LS4"
+	(label "ECU_OUT_LS4"
 		(at 73.66 95.25 0)
 		(effects
@@
 		)
 	)
-	(label "OUT_LS3"
+	(label "ECU_OUT_LS3"
 		(at 73.66 92.71 0)
 		(effects

Commit message: Autosave
Connections:
- net OUT_IGN1 renamed ECU_OUT_IGN1
- net OUT_IGN2 renamed ECU_OUT_IGN2
- net OUT_IGN5 renamed ECU_OUT_IGN5
Changed lines of the file:
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@@
 		)
 	)
-	(label "OUT_IGN2"
+	(label "ECU_OUT_IGN2"
 		(at 73.66 100.33 0)
 		(effects
@@
 		)
 	)
-	(label "OUT_IGN5"
+	(label "ECU_OUT_IGN5"
 		(at 73.66 102.87 0)
 		(effects
@@
 		)
 	)
-	(label "OUT_IGN1"
+	(label "ECU_OUT_IGN1"
 		(at 73.66 97.79 0)
 		(effects

Commit message: Autosave
Connections:
- net OUT_IGN3 renamed ECU_OUT_IGN3
- net OUT_IGN4 renamed ECU_OUT_IGN4
Changed lines of the file:
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@@
 		)
 	)
-	(label "OUT_IGN3"
+	(label "ECU_OUT_IGN3"
 		(at 73.66 105.41 0)
 		(effects
@@
 		)
 	)
-	(label "OUT_IGN4"
+	(label "ECU_OUT_IGN4"
 		(at 73.66 107.95 0)
 		(effects
