File: ECU_INTERFACE.kicad_sch (KiCad schematic)
At the start: 14 parts, among them J10 5569-16A2, J2 5569-20A2, J3 5569-06A2, J4 5569-08A2, J5 5569-18A2

Commit message: Autosave
Connections:
- net EXT_IN_SIG_RPM-: now also JP4.2 (B)
Changed lines of the file:
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@@
+	(wire
+		(pts
+			(xy 220.98 41.91) (xy 220.98 46.99)
+		)
+		(stroke
+			(width 0)
+			(type default)
+		)
+	)
 	(wire
 		(pts
@@
 		(pts
 			(xy 152.4 86.36) (xy 151.13 86.36)
+		)
+		(stroke
+			(width 0)
+			(type default)
+		)
+	)
+	(wire
+		(pts
+			(xy 223.52 41.91) (xy 220.98 41.91)
 		)
 		(stroke
@@
 	)
 	(label "EXT_IN_SIG_RPM+"
-		(at 223.52 44.45 0)
-		(effects
-			(font
+		(at 223.52 39.37 0)
+		(effects
+			(font

Commit message: Autosave
Connections:
- net EXT_IN_SIG_RPM+: now also JP1.2 (B), JP3.2 (B)
- net EXT_IN_SIG_RPM-: now also JP2.2 (B)
Changed lines of the file:
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@@
+	)
+	(junction
+		(at 220.98 41.91)
+		(diameter 0)
+		(color 0 0 0 0)
 	)
 	(junction
@@
 	)
 	(junction
+		(at 218.44 39.37)
+		(diameter 0)
+		(color 0 0 0 0)
+	)
+	(junction
 		(at 212.09 74.93)
 		(diameter 0)
@@
 	(wire
 		(pts
+			(xy 218.44 39.37) (xy 218.44 46.99)
+		)
+		(stroke
+			(width 0)
+			(type default)
+		)
+	)
+	(wire
+		(pts
 			(xy 186.69 85.09) (xy 187.96 85.09)
 		)
@@
 	(wire
 		(pts
+			(xy 223.52 39.37) (xy 218.44 39.37)
+		)
+		(stroke
+			(width 0)
+			(type default)
+		)
+	)
+	(wire
+		(pts
 			(xy 118.11 119.38) (xy 116.84 119.38)
 		)
@@
 	(wire
 		(pts
+			(xy 212.09 39.37) (xy 212.09 46.99)
+		)
+		(stroke
+			(width 0)
+			(type default)
+		)
+	)
+	(wire
+		(pts
 			(xy 119.38 114.3) (xy 118.11 114.3)
 		)
@@
 	(wire
 		(pts
+			(xy 214.63 41.91) (xy 220.98 41.91)
+		)
+		(stroke
+			(width 0)
+			(type default)
+		)
+	)
+	(wire
+		(pts
 			(xy 187.96 87.63) (xy 189.23 87.63)
 		)
@@
 	(wire
 		(pts
+			(xy 218.44 39.37) (xy 212.09 39.37)
+		)
+		(stroke
+			(width 0)
+			(type default)
+		)
+	)
+	(wire
+		(pts
 			(xy 152.4 71.12) (xy 151.13 71.12)
 		)
@@
 		)
 		(stroke
+			(width 0)
+			(type default)
+		)
+	)
+	(wire
+		(pts
+			(xy 214.63 46.99) (xy 214.63 41.91)
+		)
+		(stroke

Commit message: Autosave
Connections:
- net EXT_IN_SIG_RPM+: no longer JP1.2 (B), JP3.2 (B)
- net EXT_IN_SIG_RPM-: no longer JP2.2 (B)
Changed lines of the file:
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@@
-	)
-	(junction
-		(at 220.98 41.91)
-		(diameter 0)
-		(color 0 0 0 0)
 	)
 	(junction
@@
 	)
 	(junction
-		(at 218.44 39.37)
-		(diameter 0)
-		(color 0 0 0 0)
-	)
-	(junction
 		(at 212.09 74.93)
 		(diameter 0)
@@
 		(color 0 0 0 0)
 	)
+	(junction
+		(at 220.98 44.45)
+		(diameter 0)
+		(color 0 0 0 0)
+	)
 	(wire
 		(pts
@@
 	(wire
 		(pts
-			(xy 218.44 39.37) (xy 218.44 46.99)
-		)
-		(stroke
-			(width 0)
-			(type default)
-		)
-	)
-	(wire
-		(pts
 			(xy 186.69 85.09) (xy 187.96 85.09)
 		)
@@
 	(wire
 		(pts
-			(xy 223.52 39.37) (xy 218.44 39.37)
-		)
-		(stroke
-			(width 0)
-			(type default)
-		)
-	)
-	(wire
-		(pts
 			(xy 118.11 119.38) (xy 116.84 119.38)
 		)
@@
 	(wire
 		(pts
-			(xy 212.09 39.37) (xy 212.09 46.99)
-		)
-		(stroke
-			(width 0)
-			(type default)
-		)
-	)
-	(wire
-		(pts
 			(xy 119.38 114.3) (xy 118.11 114.3)
 		)
@@
 	(wire
 		(pts
-			(xy 220.98 41.91) (xy 220.98 46.99)
-		)
-		(stroke
-			(width 0)
-			(type default)
-		)
-	)
-	(wire
-		(pts
 			(xy 220.98 63.5) (xy 220.98 67.31)
 		)
@@
 	(wire
 		(pts
-			(xy 214.63 41.91) (xy 220.98 41.91)
+			(xy 214.63 44.45) (xy 220.98 44.45)
 		)
 		(stroke
@@
 	(wire
 		(pts
-			(xy 218.44 39.37) (xy 212.09 39.37)
+			(xy 212.09 41.91) (xy 223.52 41.91)
 		)
 		(stroke
@@
 	(wire
 		(pts
-			(xy 214.63 46.99) (xy 214.63 41.91)
-		)
-		(stroke
-			(width 0)
-			(type default)
-		)
-	)
-	(wire
-		(pts
 			(xy 212.09 63.5) (xy 212.09 74.93)
 		)
@@
 	(wire
 		(pts
+			(xy 220.98 44.45) (xy 220.98 46.99)
+		)
+		(stroke
+			(width 0)
+			(type default)
+		)
+	)
+	(wire
+		(pts
 			(xy 222.25 67.31) (xy 220.98 67.31)
 		)
@@
 	(wire
 		(pts
+			(xy 220.98 44.45) (xy 223.52 44.45)
+		)
+		(stroke
+			(width 0)
+			(type default)
+		)
+	)
+	(wire
+		(pts
 			(xy 118.11 114.3) (xy 118.11 116.84)
 		)
@@
 		(pts
 			(xy 152.4 86.36) (xy 151.13 86.36)
-		)
-		(stroke
-			(width 0)
-			(type default)
-		)
-	)
-	(wire
-		(pts
-			(xy 223.52 41.91) (xy 220.98 41.91)
 		)
 		(stroke
@@
 	)
 	(label "EXT_IN_SIG_RPM+"
-		(at 223.52 39.37 0)
+		(at 223.52 41.91 0)
 		(effects
 			(font
@@
 	)
 	(label "EXT_IN_SIG_RPM-"
-		(at 223.52 41.91 0)
-		(effects
-			(font
+		(at 223.52 44.45 0)
+		(effects
+			(font

Commit message: Autosave
Connections:
- net EXT_IN_SIG_RPM-: no longer JP4.2 (B)
Changed lines of the file:
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@@
 		(color 0 0 0 0)
 	)
-	(junction
-		(at 220.98 44.45)
-		(diameter 0)
-		(color 0 0 0 0)
-	)
 	(wire
 		(pts
@@
 	(wire
 		(pts
-			(xy 214.63 44.45) (xy 220.98 44.45)
-		)
-		(stroke
-			(width 0)
-			(type default)
-		)
-	)
-	(wire
-		(pts
 			(xy 187.96 87.63) (xy 189.23 87.63)
 		)
@@
 	(wire
 		(pts
-			(xy 212.09 41.91) (xy 223.52 41.91)
-		)
-		(stroke
-			(width 0)
-			(type default)
-		)
-	)
-	(wire
-		(pts
 			(xy 152.4 71.12) (xy 151.13 71.12)
 		)
@@
 	(wire
 		(pts
-			(xy 220.98 44.45) (xy 220.98 46.99)
-		)
-		(stroke
-			(width 0)
-			(type default)
-		)
-	)
-	(wire
-		(pts
 			(xy 222.25 67.31) (xy 220.98 67.31)
 		)
@@
 		(pts
 			(xy 222.25 72.39) (xy 214.63 72.39)
-		)
-		(stroke
-			(width 0)
-			(type default)
-		)
-	)
-	(wire
-		(pts
-			(xy 220.98 44.45) (xy 223.52 44.45)
 		)
 		(stroke
@@
 	)
 	(label "EXT_IN_SIG_RPM+"
-		(at 223.52 41.91 0)
+		(at 223.52 43.18 0)
 		(effects
 			(font
@@
 	)
 	(label "EXT_IN_SIG_RPM-"
-		(at 223.52 44.45 0)
-		(effects
-			(font
+		(at 223.52 45.72 0)
+		(effects
+			(font

Commit message: SCH Save
Connections:
- net EXT_IN_SIG_RPM+: now also JP1.2 (B), JP3.2 (B)
- net EXT_IN_SIG_RPM-: now also JP2.2 (B), JP4.2 (B)
Changed lines of the file:
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@@
+	)
+	(junction
+		(at 220.98 45.72)
+		(diameter 0)
+		(color 0 0 0 0)
 	)
 	(junction
@@
 		(color 0 0 0 0)
 	)
+	(junction
+		(at 218.44 43.18)
+		(diameter 0)
+		(color 0 0 0 0)
+	)
 	(wire
 		(pts
@@
 	(wire
 		(pts
+			(xy 212.09 43.18) (xy 218.44 43.18)
+		)
+		(stroke
+			(width 0)
+			(type default)
+		)
+	)
+	(wire
+		(pts
 			(xy 85.09 73.66) (xy 86.36 73.66)
 		)
@@
 	(wire
 		(pts
+			(xy 214.63 45.72) (xy 214.63 46.99)
+		)
+		(stroke
+			(width 0)
+			(type default)
+		)
+	)
+	(wire
+		(pts
 			(xy 186.69 85.09) (xy 187.96 85.09)
 		)
@@
 	(wire
 		(pts
+			(xy 220.98 45.72) (xy 214.63 45.72)
+		)
+		(stroke
+			(width 0)
+			(type default)
+		)
+	)
+	(wire
+		(pts
 			(xy 137.16 66.04) (xy 138.43 66.04)
 		)
@@
 	(wire
 		(pts
+			(xy 212.09 46.99) (xy 212.09 43.18)
+		)
+		(stroke
+			(width 0)
+			(type default)
+		)
+	)
+	(wire
+		(pts
 			(xy 201.93 74.93) (xy 212.09 74.93)
 		)
@@
 	(wire
 		(pts
+			(xy 220.98 45.72) (xy 220.98 46.99)
+		)
+		(stroke
+			(width 0)
+			(type default)
+		)
+	)
+	(wire
+		(pts
 			(xy 85.09 67.31) (xy 85.09 68.58)
 		)
@@
 	(wire
 		(pts
+			(xy 223.52 43.18) (xy 218.44 43.18)
+		)
+		(stroke
+			(width 0)
+			(type default)
+		)
+	)
+	(wire
+		(pts
 			(xy 102.87 121.92) (xy 104.14 121.92)
 		)
@@
 	(wire
 		(pts
+			(xy 223.52 45.72) (xy 220.98 45.72)
+		)
+		(stroke
+			(width 0)
+			(type default)
+		)
+	)
+	(wire
+		(pts
 			(xy 118.11 109.22) (xy 116.84 109.22)
 		)
@@
 		)
 		(stroke
+			(width 0)
+			(type default)
+		)
+	)
+	(wire
+		(pts
+			(xy 218.44 43.18) (xy 218.44 46.99)
+		)
+		(stroke

Commit message: Autosave
Other:
- note added: "To choose which VR to use"
Changed lines of the file:
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@@
 	(generator_version "10.0")
 	(paper "A4")
+	(rectangle
+		(start 226.06 49.53)
+		(end 247.015 58.42)
+		(stroke
+			(width 0)
+			(type default)
+		)
+		(fill
+			(type none)
+		)
+	)
 	(text "A"
 		(exclude_from_sim no)
@@
 		)
 	)
+	(text "To choose which\nVR to use"
+		(exclude_from_sim no)
+		(at 233.172 52.832 0)
+		(effects
+			(font
+				(size 1.27 1.27)
+			)
+		)
+	)

Commit message: Autosave
Other:
- note added: "To choose which VR to activate"
- note removed: "To choose which VR to use"
Changed lines of the file:
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@@
 		)
 	)
-	(text "To choose which\nVR to use"
+	(text "To choose which\nVR to activate"
 		(exclude_from_sim no)
-		(at 233.172 52.832 0)
+		(at 226.568 52.578 0)
 		(effects
 			(font
 				(size 1.27 1.27)
 			)
+			(justify left)
 		)
 	)
