File: Hub-2.0.kicad_pcb (KiCad board)
At the start: 2 copper layers, 120 x 100 mm, 17 parts, among them CN4 DT15-12PA, CN5 DT15-12PA, CN6 DT15-12PA, J10-PCB1 5569-16A2, J2-PCB1 5569-20A2, J3-PCB1 5569-06A2, J4-PCB1 5569-08A2, J5-PCB1 5569-18A2

Commit message: Autosave
Parts:
- moved J2-PCB1 171.1 mm to (51.0, 34.7)
- moved H1 171.1 mm to (43.9, 28.9)
- moved H2 171.1 mm to (43.9, 121.9)
- moved H4 171.1 mm to (136.9, 28.9)
- moved J10-PCB1 171.1 mm to (100.7, 34.7)
- moved J4-PCB1 171.1 mm to (49.7, 99.6)
- moved J5-PCB1 171.1 mm to (49.7, 80.2)
- moved CN4 164.9 mm to (146.6, 101.5)
- moved CN5 164.9 mm to (110.4, 101.5)
- moved CN6 164.9 mm to (74.4, 101.5)
Changed lines of the file:
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@@
 	(footprint "MountingHole:MountingHole_3.2mm_M3_Pad_Via"
 		(layer "F.Cu")
-		(at 212.2 -1.8)
+		(at 43.925001 28.9)
 		(descr "Mounting Hole 3.2mm, M3")
 		(tags "mounting hole 3.2mm m3")
@@
 	(footprint "MountingHole:MountingHole_3.2mm_M3_Pad_Via"
 		(layer "F.Cu")
-		(at 212.2 91.2)
+		(at 43.925001 121.9)
 		(descr "Mounting Hole 3.2mm, M3")
 		(tags "mounting hole 3.2mm m3")
@@
 	(footprint "MountingHole:MountingHole_3.2mm_M3_Pad_Via"
 		(layer "F.Cu")
-		(at 305.2 -1.8)
+		(at 136.925001 28.9)
 		(descr "Mounting Hole 3.2mm, M3")
 		(tags "mounting hole 3.2mm m3")
@@
 	(footprint "Connector_Molex:Molex_Mini-Fit_Jr_5569-16A2_2x08_P4.20mm_Horizontal"
 		(layer "F.Cu")
-		(at 269 3.975)
+		(at 100.725001 34.675)
 		(descr "Molex Mini-Fit Jr. Power Connectors, old mpn/engineering number: 5569-16A2, example for new mpn: 39-30-0160, 8 Pins per row, Mounting: Snap-in Plastic Peg PCB Lock (http://www.molex.com/pdm_docs/sd/039300020_sd.pdf)")
 		(tags "connector Molex Mini-Fit_Jr horizontalplastic_peg")
@@
 	(footprint "Connector_Molex:Molex_Mini-Fit_Jr_5569-08A2_2x04_P4.20mm_Horizontal"
 		(layer "F.Cu")
-		(at 217.975 68.9 90)
+		(at 49.700001 99.6 90)
 		(descr "Molex Mini-Fit Jr. Power Connectors, old mpn/engineering number: 5569-08A2, example for new mpn: 39-30-0080, 4 Pins per row, Mounting: Snap-in Plastic Peg PCB Lock (http://www.molex.com/pdm_docs/sd/039300020_sd.pdf)")
 		(tags "connector Molex Mini-Fit_Jr horizontalplastic_peg")
@@
 	(footprint "Connector_Molex:Molex_Mini-Fit_Jr_5569-20A2_2x10_P4.20mm_Horizontal"
 		(layer "F.Cu")
-		(at 219.3 3.975)
+		(at 51.025001 34.675)
 		(descr "Molex Mini-Fit Jr. Power Connectors, old mpn/engineering number: 5569-20A2, example for new mpn: 39-30-0200, 10 Pins per row, Mounting: Snap-in Plastic Peg PCB Lock (http://www.molex.com/pdm_docs/sd/039300020_sd.pdf)")
 		(tags "connector Molex Mini-Fit_Jr horizontalplastic_peg")
@@
 	(footprint "Connector_Molex:Molex_Mini-Fit_Jr_5569-18A2_2x09_P4.20mm_Horizontal"
 		(layer "F.Cu")
-		(at 217.95 49.55 90)
+		(at 49.675001 80.25 90)
 		(descr "Molex Mini-Fit Jr. Power Connectors, old mpn/engineering number: 5569-18A2, example for new mpn: 39-30-0180, 9 Pins per row, Mounting: Snap-in Plastic Peg PCB Lock (http://www.molex.com/pdm_docs/sd/039300020_sd.pdf)")
 		(tags "connector Molex Mini-Fit_Jr horizontalplastic_peg")
@@
 	(footprint "EasyEDA:CONN-TH_DT15-12PA"
 		(layer "B.Cu")
-		(at 267.2 152.55 180)
+		(at 110.44 101.53 180)
 		(property "Reference" "CN5"
 			(at 0 15.11 0)
@@
 	(footprint "EasyEDA:CONN-TH_DT15-12PA"
 		(layer "B.Cu")
-		(at 303.32 152.55 180)
+		(at 146.56 101.53 180)
 		(property "Reference" "CN4"
 			(at 0 15.11 0)
@@
 	(footprint "EasyEDA:CONN-TH_DT15-12PA"
 		(layer "B.Cu")
-		(at 231.2 152.55 180)
+		(at 74.44 101.53 180)
 		(property "Reference" "CN6"
 			(at 0 15.11 0)
@@
 	)
 	(gr_rect
-		(start 208.4 -5.4)
-		(end 328.4 94.6)
+		(start 40.125001 25.3)
+		(end 160.125001 125.3)
 		(stroke
 			(width 0.2)
@@
 	)
 	(gr_line
-		(start 208.7 -1.8)
-		(end 208.7 91.2)
+		(start 40.425001 28.9)
+		(end 40.425001 121.9)
 		(stroke
 			(width 0.1)
@@
 	)
 	(gr_arc
-		(start 208.7 -1.8)
-		(mid 209.725126 -4.274874)
-		(end 212.2 -5.3)
+		(start 40.425001 28.9)
+		(mid 41.450127 26.425126)
+		(end 43.925001 25.4)
 		(stroke
 			(width 0.1)
@@
 	)
 	(gr_arc
-		(start 212.2 94.7)
-		(mid 209.725126 93.674874)
-		(end 208.7 91.2)
+		(start 43.925001 125.4)
+		(mid 41.450127 124.374874)
+		(end 40.425001 121.9)
 		(stroke
 			(width 0.1)
@@
 	)
 	(gr_line
-		(start 212.2 94.7)
-		(end 305.2 94.7)
+		(start 43.925001 125.4)
+		(end 136.925001 125.4)
 		(stroke
 			(width 0.1)
@@
 	)
 	(gr_line
-		(start 305.2 -5.3)
-		(end 212.2 -5.3)
+		(start 136.925001 25.4)
+		(end 43.925001 25.4)
 		(stroke
 			(width 0.1)
@@
 	)
 	(gr_arc
-		(start 305.2 -5.3)
-		(mid 307.674874 -4.274874)
-		(end 308.7 -1.8)
+		(start 136.925001 25.4)
+		(mid 139.399875 26.425126)
+		(end 140.425001 28.9)
 		(stroke
 			(width 0.1)
@@
 	)
 	(gr_arc
-		(start 308.7 91.2)
-		(mid 307.674874 93.674874)
-		(end 305.2 94.7)
+		(start 140.425001 121.9)
+		(mid 139.399875 124.374874)
+		(end 136.925001 125.4)
 		(stroke
 			(width 0.1)
@@
 	)
 	(gr_line
-		(start 308.7 91.2)
-		(end 308.7 -1.8)
+		(start 140.425001 121.9)
+		(end 140.425001 28.9)
 		(stroke
 			(width 0.1)
@@
 	)
 	(segment
-		(start 258.62 23.715)
-		(end 258.58 23.675)
+		(start 90.345001 54.415)
+		(end 90.305001 54.375)
 		(width 0.2)
 		(layer "F.Cu")

Commit message: PCB Save
Parts:
- removed H1: M3, MountingHole:MountingHole_3.2mm_M3_Pad_Via
Changed lines of the file:
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@@
 		)
-	)
-	(footprint "MountingHole:MountingHole_3.2mm_M3_Pad_Via"
-		(layer "F.Cu")
-		(at 43.925001 28.9)
-		(descr "Mounting Hole 3.2mm, M3")
-		(tags "mounting hole 3.2mm m3")
-		(property "Reference" "H1"
-			(at 0 -4.2 0)
-			(layer "F.SilkS")
-			(hide yes)
-			(effects
-				(font
-					(size 1 1)
-					(thickness 0.15)
-				)
-			)
-		)
-		(property "Value" "M3"
-			(at 0 4.2 0)
-			(layer "F.Fab")
-			(effects
-				(font
-					(size 1 1)
-					(thickness 0.15)
-				)
-			)
-		)
-		(property "Datasheet" ""
-			(at 0 0 0)
-			(layer "F.Fab")
-			(hide yes)
-			(effects
-				(font
-					(size 1.27 1.27)
-					(thickness 0.15)
-				)
-			)
-		)
-		(property "Description" "Mounting Hole with connection"
-			(at 0 0 0)
-			(layer "F.Fab")
-			(hide yes)
-			(effects
-				(font
-					(size 1.27 1.27)
-					(thickness 0.15)
-				)
-			)
-		)
-		(property ki_fp_filters "MountingHole*Pad*")
-		(sheetname "Корневой лист")
-		(sheetfile "uaefi.kicad_sch")
-		(attr exclude_from_pos_files exclude_from_bom)
-		(duplicate_pad_numbers_are_jumpers no)
-		(fp_circle
-			(center 0 0)
-			(end 3.2 0)
-			(stroke
-				(width 0.15)
-				(type solid)
-			)
-			(fill no)
-			(layer "Cmts.User")
-		)
-		(fp_circle
-			(center 0 0)
-			(end 3.45 0)
-			(stroke
-				(width 0.05)
-				(type solid)
-			)
-			(fill no)
-			(layer "F.CrtYd")
-		)
-		(fp_text user "${REFERENCE}"
-			(at 0 0 0)
-			(layer "F.Fab")
-			(effects
-				(font
-					(size 1 1)
-					(thickness 0.15)
-				)
-			)
-		)
-		(pad "1" thru_hole circle
-			(at -2.4 0)
-			(size 0.8 0.8)
-			(drill 0.5)
-			(layers "*.Cu" "*.Mask")
-			(remove_unused_layers no)
-			(net "unconnected-(H1-Pad1)_1")
-			(pinfunction "1")
-			(pintype "input+no_connect")
-		)
-		(pad "1" thru_hole circle
-			(at -1.697056 -1.697056)
-			(size 0.8 0.8)
-			(drill 0.5)
-			(layers "*.Cu" "*.Mask")
-			(remove_unused_layers no)
-			(net "unconnected-(H1-Pad1)_8")
-			(pinfunction "1")
-			(pintype "input+no_connect")
-		)
-		(pad "1" thru_hole circle
-			(at -1.697056 1.697056)
-			(size 0.8 0.8)
-			(drill 0.5)
-			(layers "*.Cu" "*.Mask")
-			(remove_unused_layers no)
-			(net "unconnected-(H1-Pad1)_5")
-			(pinfunction "1")
-			(pintype "input+no_connect")
-		)
-		(pad "1" thru_hole circle
-			(at 0 -2.4)
-			(size 0.8 0.8)
-			(drill 0.5)
-			(layers "*.Cu" "*.Mask")
-			(remove_unused_layers no)
-			(net "unconnected-(H1-Pad1)_6")
-			(pinfunction "1")
-			(pintype "input+no_connect")
-		)
-		(pad "1" thru_hole circle
-			(at 0 0)
-			(size 6.4 6.4)
-			(drill 3.2)
-			(layers "*.Cu" "*.Mask")
-			(remove_unused_layers no)
-			(net "unconnected-(H1-Pad1)_2")
-			(pinfunction "1")
-			(pintype "input+no_connect")
-		)
-		(pad "1" thru_hole circle
-			(at 0 2.4)
-			(size 0.8 0.8)
-			(drill 0.5)
-			(layers "*.Cu" "*.Mask")
-			(remove_unused_layers no)
-			(net "unconnected-(H1-Pad1)")
-			(pinfunction "1")
-			(pintype "input+no_connect")
-		)
-		(pad "1" thru_hole circle
-			(at 1.697056 -1.697056)
-			(size 0.8 0.8)
-			(drill 0.5)
-			(layers "*.Cu" "*.Mask")
-			(remove_unused_layers no)
-			(net "unconnected-(H1-Pad1)_7")
-			(pinfunction "1")
-			(pintype "input+no_connect")
-		)
-		(pad "1" thru_hole circle
-			(at 1.697056 1.697056)
-			(size 0.8 0.8)
-			(drill 0.5)
-			(layers "*.Cu" "*.Mask")
-			(remove_unused_layers no)
-			(net "unconnected-(H1-Pad1)_3")
-			(pinfunction "1")
-			(pintype "input+no_connect")
-		)
-		(pad "1" thru_hole circle
-			(at 2.4 0)
-			(size 0.8 0.8)
-			(drill 0.5)
-			(layers "*.Cu" "*.Mask")
-			(remove_unused_layers no)
-			(net "unconnected-(H1-Pad1)_4")
-			(pinfunction "1")
-			(pintype "input+no_connect")
-		)
-		(embedded_fonts no)
 	)
 	(footprint "EasyEDA:CAP-TH_L5.5-W3.8-P5.08-D0.5"
