File: Hub-2.0.kicad_pcb (KiCad board)
At the start: 2 copper layers, 149.2 x 100 mm, 41 parts, among them CN4 DT15-12PA, CN5 DT15-12PA, CN6 DT15-12PA, J10-PCB1 5569-16A2, J2-PCB1 5569-20A2, J3-PCB1 5569-06A2, J4-PCB1 5569-08A2, J5-PCB1 5569-18A2

Commit message: Autosave
Connections:
- net /EXTERNAL_CONNECTORS/EXT_IN_SIG_COOLANT_TEMP renamed EXT_IN_SIG_COOLANT_TEMP
- net /EXTERNAL_CONNECTORS/EXT_IN_SIG_INTAKE_TEMP renamed EXT_IN_SIG_INTAKE_TEMP
- net /EXTERNAL_CONNECTORS/EXT_IN_SIG_RPM- renamed EXT_IN_SIG_RPM-
- net /EXTERNAL_CONNECTORS/EXT_IN_SIG_THROTTLE_POSITION renamed EXT_IN_SIG_THROTTLE_POSITION
- net /EXTERNAL_CONNECTORS/EXT_OUT_SIG_IGNITION renamed EXT_OUT_SIG_IGNITION
- net /EXTERNAL_CONNECTORS/EXT_OUT_SIG_INJECTOR renamed EXT_OUT_SIG_INJECTOR
Changed lines of the file:
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@@
 			(layers "*.Cu" "*.Mask")
 			(remove_unused_layers no)
-			(net "/EXTERNAL_CONNECTORS/EXT_IN_SIG_RPM-")
+			(net "EXT_IN_SIG_RPM-")
 			(pinfunction "7_7")
 			(pintype "unspecified")
@@
 			(layers "*.Cu" "*.Mask")
 			(remove_unused_layers no)
-			(net "/EXTERNAL_CONNECTORS/EXT_IN_SIG_THROTTLE_POSITION")
+			(net "EXT_IN_SIG_THROTTLE_POSITION")
 			(pinfunction "8_8")
 			(pintype "unspecified")
@@
 			(layers "*.Cu" "*.Mask")
 			(remove_unused_layers no)
-			(net "/EXTERNAL_CONNECTORS/EXT_IN_SIG_COOLANT_TEMP")
+			(net "EXT_IN_SIG_COOLANT_TEMP")
 			(pinfunction "9_9")
 			(pintype "unspecified")
@@
 			(layers "*.Cu" "*.Mask")
 			(remove_unused_layers no)
-			(net "/EXTERNAL_CONNECTORS/EXT_IN_SIG_INTAKE_TEMP")
+			(net "EXT_IN_SIG_INTAKE_TEMP")
 			(pinfunction "10_10")
 			(pintype "unspecified")
@@
 			(layers "*.Cu" "*.Mask")
 			(remove_unused_layers no)
-			(net "/EXTERNAL_CONNECTORS/EXT_OUT_SIG_INJECTOR")
+			(net "EXT_OUT_SIG_INJECTOR")
 			(pinfunction "11_11")
 			(pintype "unspecified")
@@
 			(layers "*.Cu" "*.Mask")
 			(remove_unused_layers no)
-			(net "/EXTERNAL_CONNECTORS/EXT_OUT_SIG_IGNITION")
+			(net "EXT_OUT_SIG_IGNITION")
 			(pinfunction "12_12")
 			(pintype "unspecified")

Commit message: Autosave
Connections:
- NT10 pad 1: /ECU_INTERFACE/EXT_OUT_SIG_IGNITION -> EXT_OUT_SIG_IGNITION
- NT12 pad 1: /ECU_INTERFACE/EXT_IN_SIG_COOLANT_TEMP -> EXT_IN_SIG_COOLANT_TEMP
- NT13 pad 1: /ECU_INTERFACE/EXT_IN_SIG_INTAKE_TEMP -> EXT_IN_SIG_INTAKE_TEMP
- NT7 pad 2: /ECU_INTERFACE/EXT_OUT_SIG_INJECTOR -> EXT_OUT_SIG_INJECTOR
- NT9 pad 1: /ECU_INTERFACE/EXT_IN_SIG_THROTTLE_POSITION -> EXT_IN_SIG_THROTTLE_POSITION
Changed lines of the file:
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@@
 			(size 0.5 0.5)
 			(layers "F.Cu")
-			(net "/ECU_INTERFACE/EXT_IN_SIG_INTAKE_TEMP")
+			(net "EXT_IN_SIG_INTAKE_TEMP")
 			(pinfunction "1_1")
 			(pintype "passive")
@@
 			(size 0.5 0.5)
 			(layers "F.Cu")
-			(net "/ECU_INTERFACE/EXT_OUT_SIG_INJECTOR")
+			(net "EXT_OUT_SIG_INJECTOR")
 			(pinfunction "2_2")
 			(pintype "passive")
@@
 			(size 0.5 0.5)
 			(layers "F.Cu")
-			(net "/ECU_INTERFACE/EXT_IN_SIG_THROTTLE_POSITION")
+			(net "EXT_IN_SIG_THROTTLE_POSITION")
 			(pinfunction "1_1")
 			(pintype "passive")
@@
 			(size 0.5 0.5)
 			(layers "F.Cu")
-			(net "/ECU_INTERFACE/EXT_IN_SIG_COOLANT_TEMP")
+			(net "EXT_IN_SIG_COOLANT_TEMP")
 			(pinfunction "1_1")
 			(pintype "passive")
@@
 			(size 0.5 0.5)
 			(layers "F.Cu")
-			(net "/ECU_INTERFACE/EXT_OUT_SIG_IGNITION")
+			(net "EXT_OUT_SIG_IGNITION")
 			(pinfunction "1_1")
 			(pintype "passive")

Commit message: Autosave
Parts:
- moved NT9 35.6 mm to (128.2, 87.8), turned to 180 degrees
Changed lines of the file:
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@@
 	(footprint "NetTie:NetTie-2_SMD_Pad0.5mm"
 		(layer "F.Cu")
-		(at 119.45 53.25)
+		(at 128.2 87.8 180)
 		(descr "Net tie, 2 pin, 0.5mm square SMD pads")
 		(tags "net tie")
@@
 		)
 		(property "Datasheet" ""
-			(at 0 0 0)
+			(at 0 0 180)
 			(unlocked yes)
 			(layer "F.Fab")
@@
 		)
 		(property "Description" "Net tie, 2 pins"
-			(at 0 0 0)
+			(at 0 0 180)
 			(unlocked yes)
 			(layer "F.Fab")
@@
 		)
 		(pad "1" smd circle
-			(at -0.5 0)
+			(at -0.499999 0 180)
 			(size 0.5 0.5)
 			(layers "F.Cu")
@@
 		)
 		(pad "2" smd circle
-			(at 0.5 0)
+			(at 0.499999 0 180)
 			(size 0.5 0.5)
 			(layers "F.Cu")

Commit message: Autosave
Parts:
- moved NT13 38.4 mm to (128.1, 96.7), turned to 180 degrees
Changed lines of the file:
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@@
 	(footprint "NetTie:NetTie-2_SMD_Pad0.5mm"
 		(layer "F.Cu")
-		(at 119.45 59.25)
+		(at 128.100001 96.71 180)
 		(descr "Net tie, 2 pin, 0.5mm square SMD pads")
 		(tags "net tie")
@@
 		)
 		(property "Datasheet" ""
-			(at 0 0 0)
+			(at 0 0 180)
 			(unlocked yes)
 			(layer "F.Fab")
@@
 		)
 		(property "Description" "Net tie, 2 pins"
-			(at 0 0 0)
+			(at 0 0 180)
 			(unlocked yes)
 			(layer "F.Fab")
@@
 		)
 		(pad "1" smd circle
-			(at -0.5 0)
+			(at -0.499999 0 180)
 			(size 0.5 0.5)
 			(layers "F.Cu")
@@
 		)
 		(pad "2" smd circle
-			(at 0.5 0)
+			(at 0.499999 0 180)
 			(size 0.5 0.5)
 			(layers "F.Cu")

Commit message: PCB Save
Parts:
- moved NT12 35.5 mm to (128.1, 92.2)
Changed lines of the file:
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@@
 	(footprint "NetTie:NetTie-2_SMD_Pad0.5mm"
 		(layer "F.Cu")
-		(at 119.45 57.75)
+		(at 128.1 92.2)
 		(descr "Net tie, 2 pin, 0.5mm square SMD pads")
 		(tags "net tie")

Commit message: PCB Save
Parts:
- turned NT12 to 180 degrees
Changed lines of the file:
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@@
 	(footprint "NetTie:NetTie-2_SMD_Pad0.5mm"
 		(layer "F.Cu")
-		(at 128.1 92.2)
+		(at 128.1 92.2 180)
 		(descr "Net tie, 2 pin, 0.5mm square SMD pads")
 		(tags "net tie")
@@
 		)
 		(property "Datasheet" ""
-			(at 0 0 0)
+			(at 0 0 180)
 			(unlocked yes)
 			(layer "F.Fab")
@@
 		)
 		(property "Description" "Net tie, 2 pins"
-			(at 0 0 0)
+			(at 0 0 180)
 			(unlocked yes)
 			(layer "F.Fab")
@@
 		)
 		(pad "1" smd circle
-			(at -0.5 0)
+			(at -0.499999 0 180)
 			(size 0.5 0.5)
 			(layers "F.Cu")
@@
 		)
 		(pad "2" smd circle
-			(at 0.5 0)
+			(at 0.499999 0 180)
 			(size 0.5 0.5)
 			(layers "F.Cu")

Commit message: Autosave
Routing:
- net /ECU_INTERFACE/ECU_IN_IAT: track 0.00 -> 67.7 mm
- net /ECU_INTERFACE/ECU_IN_CLT: track 0.00 -> 55.2 mm
- net /ECU_INTERFACE/ECU_IN_TPS1: track 0.00 -> 51.8 mm
Changed lines of the file:
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@@
 		(layer "User.4")
+	)
+	(segment
+		(start 127.700001 87.8)
+		(end 127.700001 53.700001)
+		(width 0.2)
+		(layer "F.Cu")
+		(net "/ECU_INTERFACE/ECU_IN_TPS1")
+	)
+	(segment
+		(start 117.525001 43.525001)
+		(end 117.525001 40.175)
+		(width 0.2)
+		(layer "F.Cu")
+		(net "/ECU_INTERFACE/ECU_IN_TPS1")
+	)
+	(segment
+		(start 127.700001 53.700001)
+		(end 117.525001 43.525001)
+		(width 0.2)
+		(layer "F.Cu")
+		(net "/ECU_INTERFACE/ECU_IN_TPS1")
+	)
+	(segment
+		(start 127.600002 95.604413)
+		(end 129.134415 94.07)
+		(width 0.2)
+		(layer "F.Cu")
+		(net "/ECU_INTERFACE/ECU_IN_IAT")
+	)
+	(segment
+		(start 130.625585 94.07)
+		(end 132.08 92.615585)
+		(width 0.2)
+		(layer "F.Cu")
+		(net "/ECU_INTERFACE/ECU_IN_IAT")
+	)
+	(segment
+		(start 129.134415 94.07)
+		(end 130.625585 94.07)
+		(width 0.2)
+		(layer "F.Cu")
+		(net "/ECU_INTERFACE/ECU_IN_IAT")
+	)
+	(segment
+		(start 130.808453 38.025)
+		(end 128.075001 38.025)
+		(width 0.2)
+		(layer "F.Cu")
+		(net "/ECU_INTERFACE/ECU_IN_IAT")
+	)
+	(segment
+		(start 128.075001 38.025)
+		(end 125.925001 40.175)
+		(width 0.2)
+		(layer "F.Cu")
+		(net "/ECU_INTERFACE/ECU_IN_IAT")
+	)
+	(segment
+		(start 132.08 39.296547)
+		(end 130.808453 38.025)
+		(width 0.2)
+		(layer "F.Cu")
+		(net "/ECU_INTERFACE/ECU_IN_IAT")
+	)
+	(segment
+		(start 127.600002 96.71)
+		(end 127.600002 95.604413)
+		(width 0.2)
+		(layer "F.Cu")
+		(net "/ECU_INTERFACE/ECU_IN_IAT")
+	)
+	(segment
+		(start 132.08 92.615585)
+		(end 132.08 39.296547)
+		(width 0.2)
+		(layer "F.Cu")
+		(net "/ECU_INTERFACE/ECU_IN_IAT")
+	)
+	(segment
+		(start 129.134415 89.62)
+		(end 130.625585 89.62)
+		(width 0.2)
+		(layer "F.Cu")
+		(net "/ECU_INTERFACE/ECU_IN_CLT")
+	)
+	(segment
+		(start 127.600001 91.154414)
+		(end 129.134415 89.62)
+		(width 0.2)
+		(layer "F.Cu")
+		(net "/ECU_INTERFACE/ECU_IN_CLT")
+	)
+	(segment
+		(start 131.68 88.565585)
+		(end 131.68 41.729999)
+		(width 0.2)
+		(layer "F.Cu")
+		(net "/ECU_INTERFACE/ECU_IN_CLT")
+	)
+	(segment
+		(start 131.68 41.729999)
+		(end 130.125001 40.175)
+		(width 0.2)
+		(layer "F.Cu")
+		(net "/ECU_INTERFACE/ECU_IN_CLT")
+	)
+	(segment
+		(start 130.625585 89.62)
+		(end 131.68 88.565585)
+		(width 0.2)
+		(layer "F.Cu")
+		(net "/ECU_INTERFACE/ECU_IN_CLT")
+	)
+	(segment
+		(start 127.600001 92.2)
+		(end 127.600001 91.154414)
+		(width 0.2)
+		(layer "F.Cu")
+		(net "/ECU_INTERFACE/ECU_IN_CLT")
 	)
 	(embedded_fonts no)

Commit message: SCH Save
Routing:
- net /ECU_INTERFACE/ECU_IN_IAT: track 67.7 -> 0.00 mm
- net /ECU_INTERFACE/ECU_IN_CLT: track 55.2 -> 0.00 mm
- net /ECU_INTERFACE/ECU_IN_TPS1: track 51.8 -> 0.00 mm
Changed lines of the file:
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@@
 		(layer "User.4")
-	)
-	(segment
-		(start 127.700001 87.8)
-		(end 127.700001 53.700001)
-		(width 0.2)
-		(layer "F.Cu")
-		(net "/ECU_INTERFACE/ECU_IN_TPS1")
-	)
-	(segment
-		(start 117.525001 43.525001)
-		(end 117.525001 40.175)
-		(width 0.2)
-		(layer "F.Cu")
-		(net "/ECU_INTERFACE/ECU_IN_TPS1")
-	)
-	(segment
-		(start 127.700001 53.700001)
-		(end 117.525001 43.525001)
-		(width 0.2)
-		(layer "F.Cu")
-		(net "/ECU_INTERFACE/ECU_IN_TPS1")
-	)
-	(segment
-		(start 127.600002 95.604413)
-		(end 129.134415 94.07)
-		(width 0.2)
-		(layer "F.Cu")
-		(net "/ECU_INTERFACE/ECU_IN_IAT")
-	)
-	(segment
-		(start 130.625585 94.07)
-		(end 132.08 92.615585)
-		(width 0.2)
-		(layer "F.Cu")
-		(net "/ECU_INTERFACE/ECU_IN_IAT")
-	)
-	(segment
-		(start 129.134415 94.07)
-		(end 130.625585 94.07)
-		(width 0.2)
-		(layer "F.Cu")
-		(net "/ECU_INTERFACE/ECU_IN_IAT")
-	)
-	(segment
-		(start 130.808453 38.025)
-		(end 128.075001 38.025)
-		(width 0.2)
-		(layer "F.Cu")
-		(net "/ECU_INTERFACE/ECU_IN_IAT")
-	)
-	(segment
-		(start 128.075001 38.025)
-		(end 125.925001 40.175)
-		(width 0.2)
-		(layer "F.Cu")
-		(net "/ECU_INTERFACE/ECU_IN_IAT")
-	)
-	(segment
-		(start 132.08 39.296547)
-		(end 130.808453 38.025)
-		(width 0.2)
-		(layer "F.Cu")
-		(net "/ECU_INTERFACE/ECU_IN_IAT")
-	)
-	(segment
-		(start 127.600002 96.71)
-		(end 127.600002 95.604413)
-		(width 0.2)
-		(layer "F.Cu")
-		(net "/ECU_INTERFACE/ECU_IN_IAT")
-	)
-	(segment
-		(start 132.08 92.615585)
-		(end 132.08 39.296547)
-		(width 0.2)
-		(layer "F.Cu")
-		(net "/ECU_INTERFACE/ECU_IN_IAT")
-	)
-	(segment
-		(start 129.134415 89.62)
-		(end 130.625585 89.62)
-		(width 0.2)
-		(layer "F.Cu")
-		(net "/ECU_INTERFACE/ECU_IN_CLT")
-	)
-	(segment
-		(start 127.600001 91.154414)
-		(end 129.134415 89.62)
-		(width 0.2)
-		(layer "F.Cu")
-		(net "/ECU_INTERFACE/ECU_IN_CLT")
-	)
-	(segment
-		(start 131.68 88.565585)
-		(end 131.68 41.729999)
-		(width 0.2)
-		(layer "F.Cu")
-		(net "/ECU_INTERFACE/ECU_IN_CLT")
-	)
-	(segment
-		(start 131.68 41.729999)
-		(end 130.125001 40.175)
-		(width 0.2)
-		(layer "F.Cu")
-		(net "/ECU_INTERFACE/ECU_IN_CLT")
-	)
-	(segment
-		(start 130.625585 89.62)
-		(end 131.68 88.565585)
-		(width 0.2)
-		(layer "F.Cu")
-		(net "/ECU_INTERFACE/ECU_IN_CLT")
-	)
-	(segment
-		(start 127.600001 92.2)
-		(end 127.600001 91.154414)
-		(width 0.2)
-		(layer "F.Cu")
-		(net "/ECU_INTERFACE/ECU_IN_CLT")
 	)
 	(embedded_fonts no)
