File: LOW_POWER_RELAYS.kicad_sch (KiCad schematic)
At the start: 4 parts, among them CN1 6437288-3, U1 YQ506-S-112 DM

Commit message: Autosave
Connections:
- net PWR_EN_FUEL_PUMP: now also D1.1 (K), R1.1, U1.85
Changed lines of the file:
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@@
 	(wire
 		(pts
-			(xy 71.12 76.2) (xy 74.93 76.2)
+			(xy 73.66 76.2) (xy 74.93 76.2)
 		)
 		(stroke
@@
 	(global_label "PWR_EN_FUEL_PUMP"
 		(shape bidirectional)
-		(at 64.77 68.58 180)
+		(at 73.66 76.2 180)
 		(fields_autoplaced yes)
 		(effects
@@
 		)
 		(property "Intersheetrefs" "${INTERSHEET_REFS}"
-			(at 42.704 68.58 0)
+			(at 51.594 76.2 0)
 			(hide yes)
 			(show_name no)
@@
 	(global_label "GND"
 		(shape bidirectional)
-		(at 59.69 76.2 180)
+		(at 62.23 88.9 180)
 		(fields_autoplaced yes)
 		(effects
@@
 		)
 		(property "Intersheetrefs" "${INTERSHEET_REFS}"
-			(at 51.8096 76.2 0)
-			(hide yes)
-			(show_name no)
+			(at 54.3496 88.9 0)
+			(hide yes)
+			(show_name no)

Commit message: Autosave
Connections:
- net PWR_12V: now also U1.30
Changed lines of the file:
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@@
+	(wire
+		(pts
+			(xy 101.6 97.79) (xy 101.6 96.52)
+		)
+		(stroke
+			(width 0)
+			(type default)
+		)
+	)
 	(wire
 		(pts
@@
 		(pts
 			(xy 91.44 76.2) (xy 86.36 76.2)
+		)
+		(stroke
+			(width 0)
+			(type default)
+		)
+	)
+	(wire
+		(pts
+			(xy 100.33 97.79) (xy 101.6 97.79)
 		)
 		(stroke
@@
 	(global_label "PWR_12V"
 		(shape bidirectional)
-		(at 68.58 54.61 0)
+		(at 100.33 97.79 180)
 		(fields_autoplaced yes)
 		(effects
@@
 				(size 1.27 1.27)
 			)
-			(justify left)
+			(justify right)
 		)
 		(property "Intersheetrefs" "${INTERSHEET_REFS}"
-			(at 80.5549 54.61 0)
-			(hide yes)
-			(show_name no)
-			(do_not_autoplace no)
-			(effects
-				(font
-					(size 1.27 1.27)
-				)
-				(justify left)
-			)
-		)
-	)
-	(global_label "PWR_EN_FUEL_PUMP"
-		(shape bidirectional)
-		(at 73.66 76.2 180)
-		(fields_autoplaced yes)
-		(effects
-			(font
-				(size 1.27 1.27)
-			)
-			(justify right)
-		)
-		(property "Intersheetrefs" "${INTERSHEET_REFS}"
-			(at 51.594 76.2 0)
+			(at 88.3551 97.79 0)
 			(hide yes)
 			(show_name no)
@@
 		)
 	)
-	(global_label "GND"
+	(global_label "PWR_EN_FUEL_PUMP"
 		(shape bidirectional)
-		(at 62.23 88.9 180)
+		(at 73.66 76.2 180)
 		(fields_autoplaced yes)
 		(effects
@@
 		)
 		(property "Intersheetrefs" "${INTERSHEET_REFS}"
-			(at 54.3496 88.9 0)
+			(at 51.594 76.2 0)
 			(hide yes)
 			(show_name no)
