File: DASH.kicad_sch (KiCad schematic)
At the start: 4 parts, among them CN5 ?, SW2 SW_SPST, SW3 SW_SPST

Commit message: Relay layout done, pinout assignments, M1 Notes, and 04 Sch Start
Parts:
- CN5: footprint (none) -> EasyEDA:CONN-TH_DT15-12PA; LCSC Part ? -> C5341788; MPN ? -> DT15-12PA; Manufacturer ? -> TE Connectivity(泰科电子)
Changed lines of the file:
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@@
 			)
 		)
-		(property "Footprint" ""
+		(property "Footprint" "EasyEDA:CONN-TH_DT15-12PA"
 			(at 68.58 62.23 0)
 			(hide yes)
@@
 			)
 		)
-		(property "Datasheet" "?"
+		(property "Datasheet" "https://www.lcsc.com/datasheet/C5341788.pdf"
 			(at 68.58 59.69 0)
 			(hide yes)
@@
 			)
 		)
-		(property "Manufacturer" "?"
+		(property "Manufacturer" "TE Connectivity(泰科电子)"
 			(at 68.58 57.15 0)
 			(hide yes)
@@
 			)
 		)
-		(property "MPN" "?"
+		(property "MPN" "DT15-12PA"
 			(at 68.58 54.61 0)
 			(hide yes)
@@
 			)
 		)
-		(property "LCSC Part" "?"
+		(property "LCSC Part" "C5341788"
 			(at 68.58 52.07 0)
 			(hide yes)
