File: ENGINE_WR450F.kicad_sch (KiCad schematic)
At the start: 6 parts, among them CN7 DT15-12PA

Commit message: High current layout work & Simulation
Parts:
- CN7: now not fitted; now left out of the parts list
Changed lines of the file:
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@@
 		(unit 1)
 		(body_style 1)
-		(exclude_from_sim no)
-		(in_bom yes)
-		(on_board yes)
-		(in_pos_files yes)
-		(dnp no)
+		(exclude_from_sim yes)
+		(in_bom no)
+		(on_board no)
+		(in_pos_files no)
+		(dnp yes)
 		(property "Reference" "CN7"
 			(at 72.39 75.438 0)
